File: KiCad/etapa_control.kicad_sch (KiCad schematic)
At the start: 0 parts

Commit message: Versió 1 de l'etapa de control quasi acabada (falta la part del micro)
Parts:
- added C1, C2, C3, C4, C5, C6: C, symbol Device:C
- added J1, J2: DE9_Pins, symbol Connector:DE9_Pins
- added U1: MAX3232, symbol Interface_UART:MAX3232
- added U2: SN65HVD230, Package_SO:SOIC-8_3.9x4.9mm_P1.27mm, symbol Interface_CAN_LIN:SN65HVD230
Connections:
- new net: C2.1, U1.1 (C1+)
- new net: C2.2, U1.3 (C1-)
- new net: C3.1, U1.4 (C2+)
- new net: C3.2, U1.5 (C2-)
- new net: C4.1, U1.2 (VS+)
- new net: C5.1, U1.6 (VS-)
- new net: C1.2, U1.16 (VCC)
- new net C1RX: U2.4 (R)
- new net C1TX: U2.1 (D)
- new net CANH: J2.7, U2.7 (CANH)
- new net CANL: J2.2, U2.6 (CANL)
- new net GND: C1.1, C4.2, C5.2, C6.2, J2.3, U1.15 (GND), U2.2 (GND), U2.8 (Rs)
- new net R1IN: J1.2, U1.13 (R1IN)
- new net RX: U1.10 (T2IN)
- new net T1OUT: J1.3, U1.14 (T1OUT)
- new net TX: U1.11 (T1IN)
- new net VCC: C6.1, U2.3 (VCC)
- no-connect marks 0 -> 1
Other:
- note added: "Transceptor CAN (equivalent al TJA1050)"
- note added: "Transceptor MAX3232"
- title: (none) -> Etapa de Control

Commit message: Canvis de pins en la botonera i els LEDs per controlar la bomba i el seu tancament. A més, eliminació del subesquema de control antic en aquesta branca
Parts:
- removed C1, C2, C3, C4, C5, C6: C, symbol Device:C
- removed J1, J2: DE9_Pins, symbol Connector:DE9_Pins
- removed U1: MAX3232, symbol Interface_UART:MAX3232
- removed U2: SN65HVD230, Package_SO:SOIC-8_3.9x4.9mm_P1.27mm, symbol Interface_CAN_LIN:SN65HVD230
Connections:
- no-connect marks 1 -> 0
Other:
- note removed: "Transceptor CAN (equivalent al TJA1050)"
- note removed: "Transceptor MAX3232"
