File: KiCad/etapa_control.kicad_sch (KiCad schematic)
At the start: 33 parts, among them J1 DE9_Pins, J2 DE9_Pins, J3 Conn_01x05, SW3 SW_Push_Dual, SW4 SW_Push, SW5 SW_Push, U20 PIC24HJ128GP502, U3 SN65HVD230, U4 MAX3232, Y1 Crystal

Commit message: Coses vàries nose
Parts:
- removed D3, D4: LED, LED_THT:LED_D3.0mm, symbol Device:LED
Connections:
- net GND: now also R8.2, R9.2
Other:
- note added: "Botonera pel funcionament dels motors"
- note added: "Control"
- note removed: "Botonera i LEDs pel funcionament dels motors"
Changed lines of the file:
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@@
 		(comment 1 "Versió 1 de l'esquemàtic de l'etapa de control")
 	)
+	(text "Control"
+		(exclude_from_sim no)
+		(at 137.668 21.59 0)
+		(effects
+			(font
+				(size 5.08 5.08)
+				(thickness 1.016)
+				(bold yes)
+			)
+		)
+	)
 	(text "Transceptor CAN\n(equivalent al TJA1050)"
 		(exclude_from_sim no)
@@
 		)
 	)
-	(text "Botonera i LEDs\npel funcionament \ndels motors"
+	(text "Botonera\npel funcionament \ndels motors"
 		(exclude_from_sim no)
 		(at 252.73 102.108 0)
@@
 	(wire
 		(pts
-			(xy 274.32 153.67) (xy 278.13 153.67)
-		)
-		(stroke
-			(width 0)
-			(type default)
-		)
-	)
-	(wire
-		(pts
 			(xy 146.05 176.53) (xy 143.51 176.53)
 		)
@@
 	(wire
 		(pts
-			(xy 261.62 130.81) (xy 266.7 130.81)
+			(xy 261.62 130.81) (xy 278.13 130.81)
 		)
 		(stroke
@@
 	(wire
 		(pts
-			(xy 262.89 153.67) (xy 266.7 153.67)
+			(xy 262.89 153.67) (xy 278.13 153.67)
 		)
 		(stroke
@@
 	(wire
 		(pts
-			(xy 274.32 130.81) (xy 278.13 130.81)
-		)
-		(stroke
-			(width 0)
-			(type default)
-		)
-	)
-	(wire
-		(pts
 			(xy 276.86 60.96) (xy 276.86 66.04)
 		)
@@
 	)
 	(symbol
-		(lib_id "Device:LED")
-		(at 270.51 153.67 180)
-		(unit 1)
-		(exclude_from_sim no)
-		(in_bom yes)
-		(on_board yes)
-		(dnp no)
-		(fields_autoplaced yes)
-		(property "Reference" "D4"
-			(at 272.0975 146.05 0)
-			(effects
-				(font
-					(size 1.27 1.27)
-				)
-			)
-		)
-		(property "Value" "LED"
-			(at 272.0975 148.59 0)
-			(effects
-				(font
-					(size 1.27 1.27)
-				)
-			)
-		)
-		(property "Footprint" "LED_THT:LED_D3.0mm"
-			(at 270.51 153.67 0)
-			(effects
-				(font
-					(size 1.27 1.27)
-				)
-				(hide yes)
-			)
-		)
-		(property "Datasheet" "~"
-			(at 270.51 153.67 0)
-			(effects
-				(font
-					(size 1.27 1.27)
-				)
-				(hide yes)
-			)
-		)
-		(property "Description" "Light emitting diode"
-			(at 270.51 153.67 0)
-			(effects
-				(font
-					(size 1.27 1.27)
-				)
-				(hide yes)
-			)
-		)
-		(property "Sim.Pins" "1=K 2=A"
-			(at 270.51 153.67 0)
-			(effects
-				(font
-					(size 1.27 1.27)
-				)
-				(hide yes)
-			)
-		)
-		(pin "1"
-		)
-		(pin "2"
-		)
-		(instances
-			(project "PROJECTE_CASTRO_RIBAS"
-				(path "/27a7fca5-115a-450a-aa60-496c314f6c0e/c7bfedf3-33ba-455f-a470-83e81ef64913"
-					(reference "D4")
-					(unit 1)
-				)
-			)
-		)
-	)
-	(symbol
 		(lib_id "Microchip_Custom:PIC24HJ128GP502")
 		(at 204.47 45.72 0)
@@
 					(unit 1)
 				)
-			)
-		)
-	)
-	(symbol
-		(lib_id "Device:LED")
-		(at 270.51 130.81 180)
-		(unit 1)
-		(exclude_from_sim no)
-		(in_bom yes)
-		(on_board yes)
-		(dnp no)
-		(fields_autoplaced yes)
-		(property "Reference" "D3"
-			(at 272.0975 123.19 0)
-			(effects
-				(font
-					(size 1.27 1.27)
-				)
-			)
-		)
-		(property "Value" "LED"
-			(at 272.0975 125.73 0)
-			(effects
-				(font
-					(size 1.27 1.27)
-				)
-			)
-		)
-		(property "Footprint" "LED_THT:LED_D3.0mm"
-			(at 270.51 130.81 0)
-			(effects
-				(font
-					(size 1.27 1.27)
-				)
-				(hide yes)
-			)
-		)
-		(property "Datasheet" "~"
-			(at 270.51 130.81 0)
-			(effects
-				(font
-					(size 1.27 1.27)
-				)
-				(hide yes)
-			)
-		)
-		(property "Description" "Light emitting diode"
-			(at 270.51 130.81 0)
-			(effects
-				(font
-					(size 1.27 1.27)
-				)
-				(hide yes)
-			)
-		)
-		(property "Sim.Pins" "1=K 2=A"
-			(at 270.51 130.81 0)
-			(effects
-				(font
-					(size 1.27 1.27)
-				)
-				(hide yes)
-			)
-		)
-		(pin "1"
-		)
-		(pin "2"
-		)
-		(instances
-			(project "PROJECTE_CASTRO_RIBAS"
-				(path "/27a7fca5-115a-450a-aa60-496c314f6c0e/c7bfedf3-33ba-455f-a470-83e81ef64913"
-					(reference "D3")
-					(unit 1)
-				)

Commit message: Ultims retocs a esquematic i layout
Parts:
- removed R8, R9: 220, Resistor_SMD:R_0805_2012Metric, symbol Device:R
