File: KiCad/control_v2.kicad_sch (KiCad schematic)
At the start: 10 parts, among them J1 DE9_Pins, J2 DE9_Pins, U1 MAX3232, U2 SN65HVD230

Commit message: Carpeta de simulacions creada i esquemàtics del MAIN borrats
Parts:
- removed C1, C2, C3, C4, C5, C6: C, symbol Device:C
- removed J1, J2: DE9_Pins, symbol Connector:DE9_Pins
- removed U1: MAX3232, symbol Interface_UART:MAX3232
- removed U2: SN65HVD230, Package_SO:SOIC-8_3.9x4.9mm_P1.27mm, symbol Interface_CAN_LIN:SN65HVD230
Connections:
- no-connect marks 1 -> 0
Other:
- note removed: "Transceptor CAN (equivalent al TJA1050)"
- note removed: "Transceptor MAX3232"

Commit message: Afegim 3 subesquemàtics a la branca main
Parts:
- added C1, C2, C3, C4, C5, C6, C8, C9: 100n, symbol Device:C
- added C10, C11: 22p, symbol Device:C
- added C7: 10u, symbol Device:C
- added J1, J2: DE9_Pins, symbol Connector:DE9_Pins
- added J3: Conn_01x05, symbol Connector_Generic:Conn_01x05
- added R1: 10k, symbol Device:R
- added R2: 120, symbol Device:R
- added R3, R4: 4.7k, symbol Device:R
- added U1: MAX3232, symbol Interface_UART:MAX3232
- added U2: SN65HVD230, Package_SO:SOIC-8_3.9x4.9mm_P1.27mm, symbol Interface_CAN_LIN:SN65HVD230
- added U3: PIC24HJ128GP502, symbol Microchip_Custom:PIC24HJ128GP502
- added Y1: Crystal, symbol Device:Crystal
Connections:
- new net: C2.1, U1.1 (C1+)
- new net: C2.2, U1.3 (C1-)
- new net: C7.1, U3.20 (VCAP)
- new net: C3.1, U1.4 (C2+)
- new net: C3.2, U1.5 (C2-)
- new net: C4.1, U1.2 (VS+)
- new net: C5.1, U1.6 (VS-)
- new net +3.3V: C1.1, C6.1, C8.2, C9.1, J3.3 (Pin_3), R1.1, R3.1, R4.1, U1.16 (VCC), U2.3 (VCC), U3.13 (VDD), U3.28 (AVDD)
- new net C1RX: U2.4 (R), U3.23 (RP12)
- new net C1TX: U2.1 (D), U3.24 (RP13)
- new net CANH: J2.7, R2.1, U2.7 (CANH)
- new net CANL: J2.2, R2.2, U2.6 (CANL)
- new net DO_control_bomba: U3.4 (RB0)
- new net DO_control_tancament: U3.5 (RB1)
- new net GND: C1.2, C10.2, C11.2, C4.2, C5.2, C6.2, C7.2, C8.1, C9.2, J1.5, J2.3, J3.2 (Pin_2), U1.15 (GND), U2.2 (GND), U2.8 (Rs), U3.19 (VSS), U3.27 (AVSS), U3.8 (VSS)
- new net MCLR: J3.1 (Pin_1), R1.2, U3.1 (MCLR)
- new net OSC_IN: C10.1, U3.9 (RA2), Y1.1
- new net OSC_OUT: C11.1, U3.10 (RA3), Y1.2
- new net PGC: J3.5 (Pin_5), U3.15 (RB6)
- new net PGD: J3.4 (Pin_4), U3.14 (RB5)
- new net PULS_START: U3.25 (RB14)
- new net PULS_STOP: U3.26 (RB15)
- new net R1IN: J1.2, U1.13 (R1IN)
- new net RX: U1.12 (R1OUT), U3.6 (RP2)
- new net SCL: R4.2, U3.17 (RB8)
- new net SDA: R3.2, U3.18 (RB9)
- new net T1OUT: J1.3, U1.14 (T1OUT)
- new net TX: U1.11 (T1IN), U3.7 (RP3)
- no-connect marks 0 -> 17
Other:
- note added: "Micro PIC24HJ128GP502"
- note added: "Oscil·lador"
- note added: "Part per programar mitjançant connexió"
- note added: "Transceptor CAN (equivalent al TJA1050)"
- note added: "Transceptor MAX3232"

Commit message: Alguns errors resolts, falten errors com canviar noms de unitats ''duplicats'', es fará en cas de que ja estigui tot bastant correcte
Connections:
- no-connect marks 17 -> 24
Changed lines of the file:
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@@
 	)
 	(no_connect
+		(at 220.98 57.15)
+	)
+	(no_connect
 		(at 31.75 92.71)
 	)
 	(no_connect
+		(at 220.98 71.12)
+	)
+	(no_connect
+		(at 220.98 59.69)
+	)
+	(no_connect
 		(at 31.75 55.88)
 	)
@@
 	)
 	(no_connect
+		(at 220.98 63.5)
+	)
+	(no_connect
+		(at 198.12 57.15)
+	)
+	(no_connect
 		(at 31.75 50.8)
 	)
@@
 	)
 	(no_connect
+		(at 198.12 67.31)
+	)
+	(no_connect
 		(at 31.75 53.34)
 	)
 	(no_connect
+		(at 198.12 54.61)
+	)
+	(no_connect
 		(at 102.87 146.05)
 	)
@@
 		(dnp no)
 		(fields_autoplaced yes)
-		(property "Reference" "#PWR02"
+		(property "Reference" "#PWR0104"
 			(at 82.55 179.07 0)
 			(effects
@@
 			(project "PROJECTE_CASTRO_RIBAS"
 				(path "/27a7fca5-115a-450a-aa60-496c314f6c0e/c7bfedf3-33ba-455f-a470-83e81ef64913"
-					(reference "#PWR02")
+					(reference "#PWR0104")
 					(unit 1)
 				)
@@
 		(dnp no)
 		(fields_autoplaced yes)
-		(property "Reference" "#PWR04"
+		(property "Reference" "#PWR0103"
 			(at 118.11 135.89 0)
 			(effects
@@
 			(project "PROJECTE_CASTRO_RIBAS"
 				(path "/27a7fca5-115a-450a-aa60-496c314f6c0e/c7bfedf3-33ba-455f-a470-83e81ef64913"
-					(reference "#PWR04")
+					(reference "#PWR0103")
 					(unit 1)
 				)
@@
 		(dnp no)
 		(fields_autoplaced yes)
-		(property "Reference" "#PWR03"
+		(property "Reference" "#PWR0102"
 			(at 118.11 143.51 0)
 			(effects
@@
 			(project "PROJECTE_CASTRO_RIBAS"
 				(path "/27a7fca5-115a-450a-aa60-496c314f6c0e/c7bfedf3-33ba-455f-a470-83e81ef64913"
-					(reference "#PWR03")
+					(reference "#PWR0102")
 					(unit 1)
 				)
@@
 		(on_board yes)
 		(dnp no)
-		(property "Reference" "#PWR01"
+		(property "Reference" "#PWR0101"
 			(at 92.71 102.87 0)
 			(effects
@@
 			(project "PROJECTE_CASTRO_RIBAS"
 				(path "/27a7fca5-115a-450a-aa60-496c314f6c0e/c7bfedf3-33ba-455f-a470-83e81ef64913"
-					(reference "#PWR01")
+					(reference "#PWR0101")
 					(unit 1)
 				)
@@
 		(dnp no)
 		(fields_autoplaced yes)
-		(property "Reference" "#PWR08"
+		(property "Reference" "#PWR0107"
 			(at 35.56 53.34 0)
 			(effects
@@
 			(project "PROJECTE_CASTRO_RIBAS"
 				(path "/27a7fca5-115a-450a-aa60-496c314f6c0e/c7bfedf3-33ba-455f-a470-83e81ef64913"
-					(reference "#PWR08")
+					(reference "#PWR0107")
 					(unit 1)
 				)
@@
 		(dnp no)
 		(fields_autoplaced yes)
-		(property "Reference" "#PWR05"
+		(property "Reference" "#PWR0106"
 			(at 82.55 73.66 0)
 			(effects
@@
 			(project "PROJECTE_CASTRO_RIBAS"
 				(path "/27a7fca5-115a-450a-aa60-496c314f6c0e/c7bfedf3-33ba-455f-a470-83e81ef64913"
-					(reference "#PWR05")
+					(reference "#PWR0106")
 					(unit 1)
 				)
@@
 		(dnp no)
 		(fields_autoplaced yes)
-		(property "Reference" "#PWR07"
+		(property "Reference" "#PWR0105"
 			(at 100.33 50.8 0)
 			(effects
@@
 			(project "PROJECTE_CASTRO_RIBAS"
 				(path "/27a7fca5-115a-450a-aa60-496c314f6c0e/c7bfedf3-33ba-455f-a470-83e81ef64913"
-					(reference "#PWR07")
+					(reference "#PWR0105")
 					(unit 1)
 				)
@@
 		(dnp no)
 		(fields_autoplaced yes)
-		(property "Reference" "#PWR06"
+		(property "Reference" "#PWR0108"
 			(at 69.85 68.58 0)
 			(effects
@@
 			(project "PROJECTE_CASTRO_RIBAS"
 				(path "/27a7fca5-115a-450a-aa60-496c314f6c0e/c7bfedf3-33ba-455f-a470-83e81ef64913"
-					(reference "#PWR06")
+					(reference "#PWR0108")
 					(unit 1)
 				)

Commit message: Petit canvi en etapa control
Connections:
- net +3.3V: now also C6.2; no longer C6.1
- net GND: now also C6.1; no longer C6.2
Other:
- moved on the sheet: C6
Changed lines of the file:
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@@
 	)
 	(junction
-		(at 100.33 53.34)
+		(at 82.55 38.1)
 		(diameter 0)
 		(color 0 0 0 0)
 	)
 	(junction
-		(at 231.14 68.58)
+		(at 100.33 53.34)
 		(diameter 0)
 		(color 0 0 0 0)
 	)
 	(junction
-		(at 82.55 41.91)
+		(at 231.14 68.58)
 		(diameter 0)
 		(color 0 0 0 0)
@@
 	(wire
 		(pts
-			(xy 236.22 72.39) (xy 231.14 72.39)
+			(xy 82.55 38.1) (xy 100.33 38.1)
 		)
 		(stroke
@@
 	(wire
 		(pts
-			(xy 208.28 78.74) (xy 210.82 78.74)
+			(xy 236.22 72.39) (xy 231.14 72.39)
 		)
 		(stroke
@@
 	(wire
 		(pts
-			(xy 58.42 151.13) (xy 62.23 151.13)
+			(xy 208.28 78.74) (xy 210.82 78.74)
 		)
 		(stroke
@@
 	(wire
 		(pts
-			(xy 196.85 41.91) (xy 198.12 41.91)
+			(xy 58.42 151.13) (xy 62.23 151.13)
 		)
 		(stroke
@@
 	(wire
 		(pts
-			(xy 214.63 123.19) (xy 217.17 123.19)
+			(xy 196.85 41.91) (xy 198.12 41.91)
 		)
 		(stroke
@@
 	(wire
 		(pts
-			(xy 184.15 30.48) (xy 177.8 30.48)
+			(xy 214.63 123.19) (xy 217.17 123.19)
 		)
 		(stroke
@@
 	(wire
 		(pts
-			(xy 93.98 41.91) (xy 100.33 41.91)
+			(xy 184.15 30.48) (xy 177.8 30.48)
 		)
 		(stroke
@@
 	(wire
 		(pts
-			(xy 82.55 41.91) (xy 82.55 48.26)
-		)
-		(stroke
-			(width 0)
-			(type default)
-		)
-	)
-	(wire
-		(pts
 			(xy 31.75 45.72) (xy 35.56 45.72)
 		)
@@
 	(wire
 		(pts
-			(xy 82.55 38.1) (xy 82.55 41.91)
+			(xy 82.55 35.56) (xy 82.55 38.1)
 		)
 		(stroke
@@
 	(wire
 		(pts
-			(xy 100.33 41.91) (xy 100.33 44.45)
-		)
-		(stroke
-			(width 0)
-			(type default)
-		)
-	)
-	(wire
-		(pts
 			(xy 220.98 68.58) (xy 231.14 68.58)
 		)
@@
 	(wire
 		(pts
-			(xy 82.55 41.91) (xy 86.36 41.91)
-		)
-		(stroke
-			(width 0)
-			(type default)
-		)
-	)
-	(wire
-		(pts
 			(xy 231.14 68.58) (xy 231.14 72.39)
 		)
@@
 	(wire
 		(pts
+			(xy 82.55 38.1) (xy 82.55 48.26)
+		)
+		(stroke
+			(width 0)
+			(type default)
+		)
+	)
+	(wire
+		(pts
 			(xy 210.82 137.16) (xy 217.17 137.16)
 		)
@@
 	(symbol
 		(lib_id "power:+3.3V")
-		(at 82.55 38.1 0)
+		(at 82.55 35.56 0)
 		(unit 1)
 		(exclude_from_sim no)
@@
 		(dnp no)
 		(property "Reference" "#PWR015"
-			(at 82.55 41.91 0)
+			(at 82.55 39.37 0)
 			(effects
 				(font
@@
 		)
 		(property "Value" "+3.3V"
-			(at 82.55 33.02 0)
+			(at 82.55 30.48 0)
 			(effects
 				(font
@@
 		)
 		(property "Footprint" ""
-			(at 82.55 38.1 0)
+			(at 82.55 35.56 0)
 			(effects
 				(font
@@
 		)
 		(property "Datasheet" ""
-			(at 82.55 38.1 0)
+			(at 82.55 35.56 0)
 			(effects
 				(font
@@
 		)
 		(property "Description" "Power symbol creates a global label with name \"+3.3V\""
-			(at 82.55 38.1 0)
+			(at 82.55 35.56 0)
 			(effects
 				(font
@@
 	(symbol
 		(lib_id "Device:C")
-		(at 90.17 41.91 90)
+		(at 100.33 41.91 180)
 		(unit 1)
 		(exclude_from_sim no)
@@
 		(fields_autoplaced yes)
 		(property "Reference" "C6"
-			(at 90.17 34.29 90)
+			(at 104.14 40.6399 0)
 			(effects
 				(font
 					(size 1.27 1.27)
 				)
+				(justify right)
 			)
 		)
 		(property "Value" "100n"
-			(at 90.17 36.83 90)
+			(at 104.14 43.1799 0)
 			(effects
 				(font
 					(size 1.27 1.27)
 				)
+				(justify right)
 			)
 		)
 		(property "Footprint" ""
-			(at 93.98 40.9448 0)
+			(at 99.3648 38.1 0)
 			(effects
 				(font
@@
 		)
 		(property "Datasheet" "~"
-			(at 90.17 41.91 0)
+			(at 100.33 41.91 0)
 			(effects
 				(font
@@
 		)
 		(property "Description" "Unpolarized capacitor"
-			(at 90.17 41.91 0)
+			(at 100.33 41.91 0)
 			(effects
 				(font
@@
 	(symbol
 		(lib_id "power:GND")
-		(at 100.33 44.45 0)
+		(at 100.33 45.72 0)
 		(unit 1)
 		(exclude_from_sim no)
@@
 		(fields_autoplaced yes)
 		(property "Reference" "#PWR0105"
-			(at 100.33 50.8 0)
+			(at 100.33 52.07 0)
 			(effects
 				(font
@@
 		)
 		(property "Value" "GND"
-			(at 100.33 49.53 0)
+			(at 100.33 50.8 0)
 			(effects
 				(font
@@
 		)
 		(property "Footprint" ""
-			(at 100.33 44.45 0)
+			(at 100.33 45.72 0)
 			(effects
 				(font
@@
 		)
 		(property "Datasheet" ""
-			(at 100.33 44.45 0)
+			(at 100.33 45.72 0)
 			(effects
 				(font
@@
 		)
 		(property "Description" "Power symbol creates a global label with name \"GND\" , ground"
-			(at 100.33 44.45 0)
+			(at 100.33 45.72 0)
 			(effects
 				(font

Commit message: Alfred penetrame porfa
Parts:
- U1: value MAX3232 -> FDC2214
Connections:
- net +3.3V: no longer U1.16 (VCC)
- net GND: no longer U1.15 (GND)
- net R1IN: no longer U1.13 (R1IN)
- net RX: no longer U1.12 (R1OUT)
- net T1OUT: no longer U1.14 (T1OUT)
- net TX: no longer U1.11 (T1IN)
- net at C2.1: no longer U1.1 (C1+)
- net at C2.2: no longer U1.3 (C1-)
- net at C3.1: no longer U1.4 (C2+)
- net at C3.2: no longer U1.5 (C2-)
- net at C4.1: no longer U1.2 (VS+)
- net at C5.1: no longer U1.6 (VS-)
Changed lines of the file:
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@@
 		(fields_autoplaced yes)
 		(property "Reference" "U1"
-			(at 84.6933 107.95 0)
+			(at 82.804 131.064 0)
 			(effects
 				(font
 					(size 1.27 1.27)
 				)
-				(justify left)
 			)
 		)
-		(property "Value" "MAX3232"
-			(at 84.6933 110.49 0)
+		(property "Value" "FDC2214"
+			(at 82.296 133.35 0)
 			(effects
 				(font
 					(size 1.27 1.27)
 				)
-				(justify left)
 			)
 		)
 		(property "Footprint" ""
-			(at 83.82 165.1 0)
-			(effects
-				(font
-					(size 1.27 1.27)
-				)
-				(justify left)
-				(hide yes)
-			)
-		)
-		(property "Datasheet" "https://datasheets.maximintegrated.com/en/ds/MAX3222-MAX3241.pdf"
-			(at 82.55 135.89 0)
+			(at 82.55 138.43 0)
 			(effects
 				(font
@@
 			)
 		)
-		(property "Description" "3.0V to 5.5V, Low-Power, up to 1Mbps, True RS-232 Transceivers Using Four 0.1μF External Capacitors"
+		(property "Datasheet" ""
+			(at 82.55 138.43 0)
+			(effects
+				(font
+					(size 1.27 1.27)
+				)
+				(hide yes)
+			)
+		)
+		(property "Description" ""
 			(at 82.55 138.43 0)
 			(effects
@@
 		(pin "9"
 		)
+		(pin "17"
+		)
 		(instances
-			(project "PROJECTE_CASTRO_RIBAS"
+			(project ""
+				(path "/27a7fca5-115a-450a-aa60-496c314f6c0e/214c85b5-e11a-40fa-b086-a325260ddb4b"
+					(reference "U1")
+					(unit 1)
+				)
 				(path "/27a7fca5-115a-450a-aa60-496c314f6c0e/c7bfedf3-33ba-455f-a470-83e81ef64913"
 					(reference "U1")

Commit message: MANTECAMANTECOSA
Parts:
- removed U1: FDC2214, symbol Interface_UART:MAX3232
- added U4: MAX3232, symbol Interface_UART:MAX3232
- renumbered U2 to U3, U3 to U5
Connections:
- net +3.3V: now also U4.16 (VCC)
- net GND: now also U4.15 (GND)
- net R1IN: now also U4.13 (R1IN)
- net RX: now also U4.12 (R1OUT)
- net T1OUT: now also U4.14 (T1OUT)
- net TX: now also U4.11 (T1IN)
- net at C2.1: now also U4.1 (C1+)
- net at C2.2: now also U4.3 (C1-)
- net at C3.1: now also U4.4 (C2+)
- net at C3.2: now also U4.5 (C2-)
- net at C4.1: now also U4.2 (VS+)
- net at C5.1: now also U4.6 (VS-)
