File: KiCad/PROJECTE_CASTRO_RIBAS.kicad_sch (KiCad schematic)
At the start: 0 parts

Commit message: Correccions dels sheets i títols fetes
Other:
- sheet ETAPA_INTERACCIO_I_COMUNICACIO renamed ETAPA_POTENCIA
- sheet ETAPA_ALIMENTACIO: file etapa_potencia.kicad_sch -> etapa_alimentacio.kicad_sch
- sheet ETAPA_CONTROL: file control_v2.kicad_sch -> etapa_control.kicad_sch
- sheet ETAPA_POTENCIA: file etapa_interaccio_i_comunicacio.kicad_sch -> etapa__potencia.kicad_sch
- note added: "POTÈNCIA"
- note removed: "INTERACCIÓ I COMUNICACIÓ"
Changed lines of the file:
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@@
-		)
-	)
-	(text "INTERACCIÓ\nI\nCOMUNICACIÓ"
-		(exclude_from_sim no)
-		(at 189.23 120.904 0)
-		(effects
-			(font
-				(size 5.08 5.08)
-				(thickness 1.016)
-				(bold yes)
-			)
 		)
 	)
@@
 		(exclude_from_sim no)
 		(at 187.96 52.07 0)
+		(effects
+			(font
+				(size 5.08 5.08)
+				(thickness 1.016)
+				(bold yes)
+			)
+		)
+	)
+	(text "POTÈNCIA"
+		(exclude_from_sim no)
+		(at 187.452 121.92 0)
 		(effects
 			(font
@@
 			(color 0 0 0 0.0000)
 		)
-		(property "Sheetname" "ETAPA_INTERACCIO_I_COMUNICACIO"
+		(property "Sheetname" "ETAPA_POTENCIA"
 			(at 146.05 94.5384 0)
 			(effects
@@
 			)
 		)
-		(property "Sheetfile" "etapa_interaccio_i_comunicacio.kicad_sch"
+		(property "Sheetfile" "etapa__potencia.kicad_sch"
 			(at 146.05 146.6346 0)
 			(effects
@@
 			)
 		)
-		(property "Sheetfile" "control_v2.kicad_sch"
+		(property "Sheetfile" "etapa_control.kicad_sch"
 			(at 146.05 78.0546 0)
 			(effects
@@
 			)
 		)
-		(property "Sheetfile" "etapa_potencia.kicad_sch"
+		(property "Sheetfile" "etapa_alimentacio.kicad_sch"
 			(at 36.83 78.0546 0)
 			(effects
