File: KiCad/PROJECTE_CASTRO_RIBAS.kicad_pcb (KiCad board)
At the start: 2 copper layers, 117.9 x 87.1 mm, 70 parts, among them J1 DE9_Pins, J2 DE9_Pins, J3 Conn_01x05, J4 Conn_01x02_Pin, K1 Fujitsu_FTR-LYAA005x, K2 Fujitsu_FTR-LYAA005x, SW3 SW_Push_Dual, SW4 SW_Push, SW5 SW_Push, U1 LM2596S-12, U2 LM1117DT-3.3, U20 PIC24HJ128GP502, U3 SN65HVD230, U4 MAX3232, U6 FDC2214, Y1 Crystal

Commit message: Coses vàries nose
Parts:
- removed D3, D4: LED, LED_THT:LED_D3.0mm
Connections:
- R8 pad 2: Net-(D3-A) -> GND
- R9 pad 2: Net-(D4-A) -> GND
Routing:
- net GND: track 159.5 -> 148.4 mm, vias 44 -> 43
- net Net-(D4-A): track 9.29 -> 0.00 mm
- net Net-(D3-A): track 7.30 -> 0.00 mm

Commit message: Ultims retocs a esquematic i layout
Parts:
- removed R8, R9: 220, Resistor_SMD:R_0805_2012Metric
Routing:
- net DO_control_bomba: track 78.6 -> 65.4 mm
- net GND: track 148.4 -> 137.3 mm
